File: Hardware/KiCAD/Version 1/Version 1.kicad_sch (KiCad schematic)
At the start: 6 parts

Commit message: pcb progress
Parts:
- added J1, J2, J3, J4, J5: Conn_01x03_Pin, Connector_PinHeader_2.54mm:PinHeader_1x03_P2.54mm_Vertical, symbol Connector:Conn_01x03_Pin
- added R1, R2, R3, R4, R5: 10K, Resistor_THT:R_Axial_DIN0204_L3.6mm_D1.6mm_P7.62mm_Horizontal, symbol Device:R
- added SW1: Button 1, Button_Switch_Keyboard:SW_Cherry_MX_1.00u_PCB, symbol Switch:SW_Push
- added SW2: Button 2, Button_Switch_Keyboard:SW_Cherry_MX_1.00u_PCB, symbol Switch:SW_Push
- added SW3: Button 3, Button_Switch_Keyboard:SW_Cherry_MX_1.00u_PCB, symbol Switch:SW_Push
- added SW4: Button 4, Button_Switch_Keyboard:SW_Cherry_MX_1.00u_PCB, symbol Switch:SW_Push
- added SW5: Button 5, Button_Switch_Keyboard:SW_Cherry_MX_1.00u_PCB, symbol Switch:SW_Push
Connections:
- net +5V: now also SW1.1, SW2.1, SW3.1, SW4.1, SW5.1
- net GND: now also J1.3 (Pin_3), J2.3 (Pin_3), J3.3 (Pin_3), J4.3 (Pin_3), J5.3 (Pin_3), R1.1, R2.1, R3.1, R4.1, R5.1
- net at A1.10 (D7): now also J5.2 (Pin_2)
- net at A1.11 (D8): now also J4.2 (Pin_2)
- net at A1.12 (D9): now also J3.2 (Pin_2)
- net at A1.13 (D10): now also J2.2 (Pin_2)
- net at A1.14 (MOSI): now also J1.2 (Pin_2)
- net at A1.5 (D2): now also R5.2, SW5.2
- net at A1.6 (D3): now also R4.2, SW4.2
- net at A1.7 (D4): now also R1.2, SW3.2
- net at A1.8 (D5): now also R2.2, SW2.2
- net at A1.9 (D6): now also R3.2, SW1.2
Other:
- moved on the sheet: A1, Slider1, Slider2, Slider3, Slider4, Slider5

Commit message: some more KiCAD Stuff
Other:
- moved on the sheet: A1, J1, J2, J3, J4, J5, R1, R2, R3, R4, R5, SW1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

Commit message: more kicad stuff
Parts:
- added J10, J11, J12, J13, J14, J15, J16, J6, J7, J8, J9: Conn_01x03_Pin, Connector_PinHeader_2.54mm:PinHeader_1x03_P2.54mm_Vertical, symbol Connector:Conn_01x03_Pin
- added J17: Conn_01x02_Pin, Connector_PinHeader_2.54mm:PinHeader_1x02_P2.54mm_Vertical, symbol Connector:Conn_01x02_Pin
- added U1, U2, U3, U4, U5: ~, custom_library:Custom LED Strip, symbol custom_library:Custom_LED_Strip_5V_Cob
- added U6, U7, U8: ~, custom_library:Custom Spin Potentiometer, symbol custom_library:Custom_10K_Ohm_Spin_Potentiometer
Connections:
- net +5V: now also J6.3 (Pin_3), J7.3 (Pin_3), J8.3 (Pin_3)
- net GND: now also J6.1 (Pin_1), J7.1 (Pin_1), J8.1 (Pin_1)
- net at A1.24 (SCL/A5): now also J8.2 (Pin_2)
- net at A1.25 (A6): now also J7.2 (Pin_2)
- net at A1.26 (A7): now also J6.2 (Pin_2)
- new net: J10.1 (Pin_1), J11.1 (Pin_1), J12.1 (Pin_1), J13.1 (Pin_1), J17.2 (Pin_2), J9.1 (Pin_1), U1.1 (+5V), U2.1 (+5V), U3.1 (+5V), U4.1 (+5V), U5.1 (+5V)
- new net: J10.3 (Pin_3), J11.3 (Pin_3), J12.3 (Pin_3), J13.3 (Pin_3), J17.1 (Pin_1), J9.3 (Pin_3), U1.2 (GND), U2.2 (GND), U3.2 (GND), U4.2 (GND), U5.2 (GND)
- new net: J11.2 (Pin_2), U3.3 (Data)
- new net: J10.2 (Pin_2), U2.3 (Data)
- new net: J16.1 (Pin_1), U8.1 (+5V)
- new net: J16.2 (Pin_2), U8.3 (Data)
- new net: J16.3 (Pin_3), U8.2 (GND)
- new net: J15.1 (Pin_1), U7.1 (+5V)
- new net: J15.2 (Pin_2), U7.3 (Data)
- new net: J15.3 (Pin_3), U7.2 (GND)
- new net: J13.2 (Pin_2), U5.3 (Data)
- new net: J9.2 (Pin_2), U1.3 (Data)
- new net: J12.2 (Pin_2), U4.3 (Data)
- new net: J14.1 (Pin_1), U6.1 (+5V)
- new net: J14.2 (Pin_2), U6.3 (Data)
- new net: J14.3 (Pin_3), U6.2 (GND)

Commit message: ready to order maybe
Parts:
- removed J10, J11, J12, J13, J14, J15, J16, J9: Conn_01x03_Pin, Connector_PinHeader_2.54mm:PinHeader_1x03_P2.54mm_Vertical, symbol Connector:Conn_01x03_Pin
- removed J17: Conn_01x02_Pin, Connector_PinHeader_2.54mm:PinHeader_1x02_P2.54mm_Vertical, symbol Connector:Conn_01x02_Pin
- removed U1, U2, U3, U4, U5: ~, custom_library:Custom LED Strip, symbol custom_library:Custom_LED_Strip_5V_Cob
- removed U6, U7, U8: ~, custom_library:Custom Spin Potentiometer, symbol custom_library:Custom_10K_Ohm_Spin_Potentiometer
