File: Hardware/KiCAD/Version 1/Version 1.kicad_pcb (KiCad board)
At the start: 2 copper layers, 95 x 98 mm, 6 parts

Commit message: pcb progress
Parts:
- added J1: Conn_01x03_Pin, Connector_PinHeader_2.54mm:PinHeader_1x03_P2.54mm_Vertical, F.Cu at (62.0, 65.0)
- added J2: Conn_01x03_Pin, Connector_PinHeader_2.54mm:PinHeader_1x03_P2.54mm_Vertical, F.Cu at (83.5, 65.0)
- added J3: Conn_01x03_Pin, Connector_PinHeader_2.54mm:PinHeader_1x03_P2.54mm_Vertical, F.Cu at (102.8, 65.0)
- added J4: Conn_01x03_Pin, Connector_PinHeader_2.54mm:PinHeader_1x03_P2.54mm_Vertical, F.Cu at (121.2, 65.0)
- added J5: Conn_01x03_Pin, Connector_PinHeader_2.54mm:PinHeader_1x03_P2.54mm_Vertical, F.Cu at (140.5, 65.0)
- added R1: 10K, Resistor_THT:R_Axial_DIN0204_L3.6mm_D1.6mm_P7.62mm_Horizontal, F.Cu at (102.8, 114.9)
- added R2: 10K, Resistor_THT:R_Axial_DIN0204_L3.6mm_D1.6mm_P7.62mm_Horizontal, F.Cu at (83.5, 114.7)
- added R3: 10K, Resistor_THT:R_Axial_DIN0204_L3.6mm_D1.6mm_P7.62mm_Horizontal, F.Cu at (62.0, 114.9)
- added R4: 10K, Resistor_THT:R_Axial_DIN0204_L3.6mm_D1.6mm_P7.62mm_Horizontal, F.Cu at (121.5, 115.0)
- added R5: 10K, Resistor_THT:R_Axial_DIN0204_L3.6mm_D1.6mm_P7.62mm_Horizontal, F.Cu at (140.8, 114.9)
- added SW1: Button 1, Button_Switch_Keyboard:SW_Cherry_MX_1.00u_PCB, F.Cu at (61.8, 128.4)
- added SW2: Button 2, Button_Switch_Keyboard:SW_Cherry_MX_1.00u_PCB, F.Cu at (83.3, 128.4)
- added SW3: Button 3, Button_Switch_Keyboard:SW_Cherry_MX_1.00u_PCB, F.Cu at (102.3, 128.4)
- added SW4: Button 4, Button_Switch_Keyboard:SW_Cherry_MX_1.00u_PCB, F.Cu at (121.3, 128.4)
- added SW5: Button 5, Button_Switch_Keyboard:SW_Cherry_MX_1.00u_PCB, F.Cu at (140.3, 128.4)
- A1: moved to B.Cu
- moved Slider1 25.5 mm to (49.9, 63.2)
- moved Slider2 19.1 mm to (71.4, 63.2)
- moved Slider3 15.0 mm to (90.6, 63.2)
- moved A1 13.0 mm to (91.1, 61.2)
- moved Slider4 11.4 mm to (109.4, 63.2)
- moved Slider5 7.66 mm to (128.6, 63.2)
Connections:
- A1 pad 10: unconnected-(A1-D7-Pad10) -> Net-(A1-D7)
- A1 pad 11: unconnected-(A1-D8-Pad11) -> Net-(A1-D8)
- A1 pad 12: unconnected-(A1-D9-Pad12) -> Net-(A1-D9)
- A1 pad 13: unconnected-(A1-D10-Pad13) -> Net-(A1-D10)
- A1 pad 14: unconnected-(A1-MOSI-Pad14) -> Net-(A1-MOSI)
- A1 pad 5: unconnected-(A1-D2-Pad5) -> Net-(A1-D2)
- A1 pad 6: unconnected-(A1-D3-Pad6) -> Net-(A1-D3)
- A1 pad 7: unconnected-(A1-D4-Pad7) -> Net-(A1-D4)
- A1 pad 8: unconnected-(A1-D5-Pad8) -> Net-(A1-D5)
- A1 pad 9: unconnected-(A1-D6-Pad9) -> Net-(A1-D6)
Routing:
- net GND: track 95.9 -> 250.9 mm
- net Net-(A1-D2): track 0.00 -> 99.4 mm
- net Net-(A1-D3): track 0.00 -> 90.3 mm
- net Net-(A1-D4): track 0.00 -> 83.7 mm
- net Net-(A1-D7): track 0.00 -> 79.2 mm
- net Net-(A1-D5): track 0.00 -> 78.8 mm
- net Net-(A1-D6): track 0.00 -> 76.1 mm
- net Net-(A1-D8): track 0.00 -> 60.2 mm
- net Net-(A1-A0): track 34.7 -> 82.6 mm
- net Net-(A1-D9): track 0.00 -> 44.3 mm
- net +5V: track 154.2 -> 196.9 mm
- net Net-(A1-A1): track 30.5 -> 62.1 mm
- net Net-(A1-D10): track 0.00 -> 27.6 mm
- net Net-(A1-SDA/A4): track 49.8 -> 25.9 mm
- net Net-(A1-A3): track 40.0 -> 23.9 mm, vias 0 -> 1
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Other:
- board size 95 x 98 mm -> 99 x 99 mm

Commit message: some more KiCAD Stuff
Parts:
- moved A1 20.7 mm to (105.1, 46.0), turned to -90 degrees
Routing:
- net Net-(A1-A0): track 82.6 -> 6.86 mm
- net Net-(A1-MOSI): track 8.57 -> 82.5 mm
- net Net-(A1-SDA/A4): track 25.9 -> 78.7 mm
- net Net-(A1-D7): track 79.2 -> 28.6 mm
- net Net-(A1-A1): track 62.1 -> 14.4 mm
- net Net-(A1-D6): track 76.1 -> 121.5 mm, vias 0 -> 1
- net Net-(A1-D8): track 60.2 -> 21.8 mm
- net Net-(A1-D10): track 27.6 -> 57.7 mm
- net Net-(A1-D5): track 78.8 -> 108.6 mm, vias 0 -> 1
- net Net-(A1-A3): track 23.9 -> 47.9 mm, vias 1 -> 0
- net +5V: track 196.9 -> 174.5 mm
- net Net-(A1-D4): track 83.7 -> 98.5 mm
- net Net-(A1-A2): track 39.6 -> 30.6 mm, vias 1 -> 0
- net Net-(A1-D9): track 44.3 -> 39.4 mm, vias 0 -> 1
- net GND: track 250.9 -> 248.0 mm
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
Commit message: more kicad stuff
Parts:
- added J10: Conn_01x03_Pin, Connector_PinHeader_2.54mm:PinHeader_1x03_P2.54mm_Vertical, F.Cu at (183.2, 85.0)
- added J11: Conn_01x03_Pin, Connector_PinHeader_2.54mm:PinHeader_1x03_P2.54mm_Vertical, F.Cu at (202.2, 85.0)
- added J12: Conn_01x03_Pin, Connector_PinHeader_2.54mm:PinHeader_1x03_P2.54mm_Vertical, F.Cu at (221.0, 85.0)
- added J13: Conn_01x03_Pin, Connector_PinHeader_2.54mm:PinHeader_1x03_P2.54mm_Vertical, F.Cu at (240.0, 85.0)
- added J14: Conn_01x03_Pin, Connector_PinHeader_2.54mm:PinHeader_1x03_P2.54mm_Vertical, F.Cu at (156.0, 76.5)
- added J15: Conn_01x03_Pin, Connector_PinHeader_2.54mm:PinHeader_1x03_P2.54mm_Vertical, F.Cu at (151.8, 80.8)
- added J16: Conn_01x03_Pin, Connector_PinHeader_2.54mm:PinHeader_1x03_P2.54mm_Vertical, F.Cu at (151.8, 71.5)
- added J17: Conn_01x02_Pin, Connector_PinHeader_2.54mm:PinHeader_1x02_P2.54mm_Vertical, F.Cu at (241.8, 71.0)
- added J6: Conn_01x03_Pin, Connector_PinHeader_2.54mm:PinHeader_1x03_P2.54mm_Vertical, F.Cu at (51.8, 60.8)
- added J7: Conn_01x03_Pin, Connector_PinHeader_2.54mm:PinHeader_1x03_P2.54mm_Vertical, F.Cu at (51.8, 51.5)
- added J8: Conn_01x03_Pin, Connector_PinHeader_2.54mm:PinHeader_1x03_P2.54mm_Vertical, F.Cu at (56.0, 56.5)
- added J9: Conn_01x03_Pin, Connector_PinHeader_2.54mm:PinHeader_1x03_P2.54mm_Vertical, F.Cu at (161.2, 85.0)
- added U1: ~, custom_library:Custom LED Strip, F.Cu at (158.0, 89.0)
- added U2: ~, custom_library:Custom LED Strip, F.Cu at (180.0, 89.0)
- added U3: ~, custom_library:Custom LED Strip, F.Cu at (199.0, 89.0)
- added U4: ~, custom_library:Custom LED Strip, F.Cu at (218.0, 89.0)
- added U5: ~, custom_library:Custom LED Strip, F.Cu at (237.0, 89.0)
- added U6: ~, custom_library:Custom Spin Potentiometer, F.Cu at (167.0, 70.2)
- added U7: ~, custom_library:Custom Spin Potentiometer, F.Cu at (192.8, 70.2)
- added U8: ~, custom_library:Custom Spin Potentiometer, F.Cu at (218.5, 70.2)
- moved J1 0.71 mm to (61.2, 65.0)
- moved Slider1 0.62 mm to (49.2, 63.2)
- moved J3 0.50 mm to (102.2, 65.0)
- moved J5 0.50 mm to (140.0, 65.0)
- moved Slider3 0.38 mm to (90.2, 63.2)
- moved Slider5 0.38 mm to (128.2, 63.2)
- moved J2 0.25 mm to (83.2, 65.0)
- moved J4 0.22 mm to (121.0, 65.0)
- moved Slider2 0.12 mm to (71.2, 63.2)
- moved Slider4 0.12 mm to (109.2, 63.2)
Connections:
- A1 pad 24: unconnected-(A1-SCL/A5-Pad24) -> Net-(A1-SCL/A5)
- A1 pad 25: unconnected-(A1-A6-Pad25) -> Net-(A1-A6)
- A1 pad 26: unconnected-(A1-A7-Pad26) -> Net-(A1-A7)
Routing:
- net Net-(J10-Pin_1): track 0.00 -> 259.6 mm
- net Net-(J10-Pin_3): track 0.00 -> 232.2 mm
- net +5V: track 174.5 -> 258.3 mm
- net Net-(A1-A7): track 0.00 -> 79.4 mm
- net Net-(J16-Pin_3): track 0.00 -> 78.6 mm
- net Net-(J16-Pin_2): track 0.00 -> 74.1 mm
- net Net-(A1-A6): track 0.00 -> 71.3 mm
- net Net-(J16-Pin_1): track 0.00 -> 69.5 mm
- net Net-(A1-SCL/A5): track 0.00 -> 68.4 mm
- net Net-(J15-Pin_3): track 0.00 -> 56.2 mm
- net Net-(J15-Pin_2): track 0.00 -> 50.3 mm
- net Net-(J15-Pin_1): track 0.00 -> 45.4 mm
- net Net-(J14-Pin_3): track 0.00 -> 22.9 mm
- net GND: track 248.0 -> 268.4 mm
- net Net-(J14-Pin_2): track 0.00 -> 18.5 mm
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- added copper zone on B.Cu, net GND
Other:
- board size 99 x 99 mm -> 199 x 99 mm

Commit message: ready to order maybe
Other:
- outline, holes or cut-outs redrawn
Changed lines of the file:
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@@
 		(tags "Through hole pin header THT 1x03 2.54mm single row")
 		(property "Reference" "J16"
-			(at 0 8 360)
+			(at 0 8 0)
 			(layer "F.SilkS")
 			(effects
@@
 		)
 		(property "Value" "Conn_01x03_Pin"
-			(at 0 7.41 360)
+			(at 0 7.41 0)
 			(layer "F.Fab")
 			(hide yes)
@@
 		)
 		(fp_text user "${REFERENCE}"
-			(at 0 2.54 360)
+			(at 0 2.54 0)
 			(layer "F.Fab")
 			(effects
@@
 		)
 		(fp_text user "${REFERENCE}"
-			(at 0 2.54 360)
+			(at 0 2.54 0)
 			(layer "F.Fab")
 			(effects
@@
 		(tags "Through hole pin header THT 1x03 2.54mm single row")
 		(property "Reference" "J14"
-			(at 0 -2.33 360)
+			(at 0 -2.33 0)
 			(layer "F.SilkS")
 			(effects
@@
 		)
 		(property "Value" "Conn_01x03_Pin"
-			(at 0 7.41 360)
+			(at 0 7.41 0)
 			(layer "F.Fab")
 			(hide yes)
@@
 		)
 		(fp_text user "${REFERENCE}"
-			(at 0 2.54 360)
+			(at 0 2.54 0)
 			(layer "F.Fab")
 			(effects
@@
 		(tags "Through hole pin header THT 1x03 2.54mm single row")
 		(property "Reference" "J15"
-			(at 0 -2.33 360)
+			(at 0 -2.33 0)
 			(layer "F.SilkS")
 			(effects
@@
 		)
 		(property "Value" "Conn_01x03_Pin"
-			(at 0 7.41 360)
+			(at 0 7.41 0)
 			(layer "F.Fab")
 			(hide yes)
@@
 		)
 		(fp_text user "${REFERENCE}"
-			(at 0 2.54 360)
+			(at 0 2.54 0)
 			(layer "F.Fab")
 			(effects
@@
 		)
 		(fp_text user "${REFERENCE}"
-			(at 0 2.54 360)
+			(at 0 2.54 0)
 			(layer "F.Fab")
 			(effects
@@
 	)
 	(gr_rect
+		(start 147.5 113.5)
+		(end 148.5 140.75)
+		(stroke
+			(width 0.05)
+			(type default)
+		)
+		(fill none)
+		(layer "Edge.Cuts")
+	)
+	(gr_rect
 		(start 231.75 85.75)
 		(end 234.75 140.75)
@@
 	)
 	(gr_rect
+		(start 147.5 46.75)
+		(end 148.5 74)
+		(stroke
+			(width 0.05)
+			(type default)
+		)
+		(fill none)
+		(layer "Edge.Cuts")
+	)
+	(gr_rect
 		(start 193.75 85.75)
 		(end 196.75 140.75)
@@
 	)
 	(gr_rect
-		(start 174.75 85.75)
-		(end 177.75 140.75)
+		(start 147.5 76.5)
+		(end 148.5 111)
 		(stroke
 			(width 0.05)
@@
 	)
 	(gr_rect
-		(start 148.5 44.25)
-		(end 247.5 143.25)
+		(start 174.75 85.75)
+		(end 177.75 140.75)
 		(stroke
-			(width 0.1)
+			(width 0.05)
 			(type default)
 		)
@@
 	(gr_rect
 		(start 48.5 44.25)
-		(end 147.5 143.25)
+		(end 247.5 143.25)
 		(stroke
 			(width 0.1)

Commit message: to be ordererd
Routing:
- net Net-(J10-Pin_1): track 259.6 -> 263.9 mm
- net Net-(J9-Pin_2): track 6.11 -> 6.97 mm
- net Net-(J10-Pin_2): track 6.11 -> 6.97 mm
- net Net-(J13-Pin_2): track 6.01 -> 6.86 mm
- net Net-(J11-Pin_2): track 6.11 -> 6.82 mm
